Commit message: rename the folders

File: rr_description/urdf/augmented_rc_car.urdf.xacro (robot description, xacro)
@@ -293,5 +293,5 @@
       <origin xyz="0.0 0.0 0.0" rpy="0.0 0.0 0.0"/>
       <geometry>
-        <mesh filename="package://rr_vehicle_description/urdf/RR2018.stl" scale="0.02 0.02 0.02"/>
+        <mesh filename="package://rr_description/urdf/RR2018.stl" scale="0.02 0.02 0.02"/>
       </geometry>
     </visual>

Commit message: add the asphalt ground and the autorally track

File: rr_description/urdf/augmented_rc_car.urdf.xacro (robot description, xacro)
@@ -293,5 +293,5 @@
       <origin xyz="0.0 0.0 0.0" rpy="0.0 0.0 0.0"/>
       <geometry>
-        <mesh filename="package://rr_description/urdf/RR2018.stl" scale="0.02 0.02 0.02"/>
+        <mesh filename="package://rr_description/urdf/assets/RR2018.stl" scale="0.02 0.02 0.02"/>
       </geometry>
     </visual>

Commit message: stopped the strange rolling

File: rr_description/urdf/augmented_rc_car.urdf.xacro (robot description, xacro)
@@ -139,4 +139,5 @@
       <axis xyz="0 0 -1"/>
       <limit effort="${axle_eff_limit}" velocity="${axle_vel_limit}"/>
+      <dynamics damping="0.001" friction="0.5"/>
     </joint>
     <transmission name="${lr_prefix}_${fr_prefix}_axle_trans">
@@ -146,4 +147,6 @@
       </joint>
       <actuator name="${lr_prefix}_${fr_prefix}_axle_act">
+        <!-- This hardwareInterface element exists for compatibility
+             with ROS Hydro. -->
         <hardwareInterface>EffortJointInterface</hardwareInterface>
         <mechanicalReduction>1</mechanicalReduction>
@@ -173,11 +176,10 @@
           inner_rad="${hub_dia / 2}" outer_rad="${tire_dia / 2}"
           height="${tire_width}" mass="${wheel_mass}"/>
+      <max_contacts>1</max_contacts>
     </link>
     <gazebo reference="${lr_prefix}_${fr_prefix}_wheel">
       <material>Gazebo/Black</material>
-      <kp>100000.0</kp>
-      <kd>1</kd>
-      <mu1>1.35</mu1>
-      <mu2>1.35</mu2>
+      <mu1>0.7</mu1>
+      <mu2>0.75</mu2>
       <fdir1>1 0 0</fdir1>
     </gazebo>
@@ -293,5 +295,5 @@
       <origin xyz="0.0 0.0 0.0" rpy="0.0 0.0 0.0"/>
       <geometry>
-        <mesh filename="package://rr_description/urdf/assets/RR2018.stl" scale="0.02 0.02 0.02"/>
+        <mesh filename="package://rr_description/urdf/assets/RR2018.stl" scale="0.0254 0.0254 0.0254"/>
       </geometry>
     </visual>
@@ -300,5 +302,5 @@
     <parent link="chassis"/>
     <child link="outer_shell"/>
-    <origin xyz="-0.26 -0.11 0.05" rpy="${degrees_90} 0.0 ${degrees_90}"/>
+    <origin xyz="-0.26 -0.11 0.02" rpy="${degrees_90} 0.0 ${degrees_90}"/>
   </joint>
   <!-- Wheels -->

Commit message: add drag race visual

File: rr_description/urdf/augmented_rc_car.urdf.xacro (robot description, xacro)
@@ -24,5 +24,5 @@
  -  @competition IARRC 2018
 -->
-<robot name="" xmlns:xacro="http://www.ros.org/wiki/xacro">
+<robot name="rr_platform" xmlns:xacro="http://www.ros.org/wiki/xacro">
   <!-- Degree-to-radian conversions -->
   <xacro:property name="degrees_45" value="0.785398163"/>
@@ -91,9 +91,9 @@
       <xacro:insert_block name="origin"/>
       <mass value="${mass}"/>
-      <inertia ixx="${mass * (depth * depth + height * height) / 12}"
+      <inertia ixx="${mass * (depth * depth + height * height) / 12.0}"
                ixy="0" ixz="0"
-               iyy="${mass * (width * width + height * height) / 12}"
+               iyy="${mass * (width * width + height * height) / 12.0}"
                iyz="0"
-               izz="${mass * (width * width + depth * depth) / 12}"/>
+               izz="${mass * (width * width + depth * depth) / 12.0}"/>
     </inertial>
   </xacro:macro>
@@ -105,12 +105,12 @@
     <inertial>
       <mass value="${mass}"/>
-      <inertia ixx="${(1 / 12) * mass * (3 * (inner_rad * inner_rad +
+      <inertia ixx="${(1 / 12.0) * mass * (3.0 * (inner_rad * inner_rad +
                     outer_rad * outer_rad) + height * height)}"
                ixy="0" ixz="0"
-               iyy="${(1 / 12) * mass * (3 * (inner_rad * inner_rad +
+               iyy="${(1 / 12.0) * mass * (3.0 * (inner_rad * inner_rad +
                     outer_rad * outer_rad) + height * height)}"
                iyz="0"
                izz="${mass * (inner_rad * inner_rad +
-                    outer_rad * outer_rad) / 2}"/>
+                    outer_rad * outer_rad) / 2.0}"/>
     </inertial>
   </xacro:macro>
@@ -121,6 +121,6 @@
       <parent link="chassis"/>
       <child link="${child}"/>
-      <origin xyz="${fr_reflect * wheelbase / 2}
-                   ${lr_reflect * ((hex_hub_dist / 2) - axle_length)}
+      <origin xyz="${fr_reflect * wheelbase / 2.0}
+                   ${lr_reflect * ((hex_hub_dist / 2.0) - axle_length)}
                    0"/>
     </joint>
@@ -160,5 +160,5 @@
                      0"/>
         <geometry>
-          <cylinder radius="${tire_dia / 2}" length="${tire_width}"/>
+          <cylinder radius="${tire_dia / 2.0}" length="${tire_width}"/>
         </geometry>
         <material name="tire_mat"/>
@@ -170,11 +170,23 @@
                      0"/>
         <geometry>
-          <cylinder radius="${tire_dia / 2}" length="${tire_width}"/>
+          <cylinder radius="${tire_dia / 2.0}" length="${tire_width}"/>
         </geometry>
       </collision>
       <xacro:thick_walled_tube_inertial
-          inner_rad="${hub_dia / 2}" outer_rad="${tire_dia / 2}"
+          inner_rad="${hub_dia / 2.0}" outer_rad="${tire_dia / 2.0}"
           height="${tire_width}" mass="${wheel_mass}"/>
       <max_contacts>1</max_contacts>
+      <surface>
+        <contact>
+          <ode>
+            <soft_cfm>0.000000001</soft_cfm>
+            <soft_erp>0.2</soft_erp>
+            <kp>1e+10</kp>
+            <kd>10</kd>
+            <max_vel>0.01</max_vel>
+            <min_depth>0.005</min_depth>
+          </ode>
+        </contact>
+      </surface>
     </link>
     <gazebo reference="${lr_prefix}_${fr_prefix}_wheel">
@@ -182,5 +194,4 @@
       <mu1>0.7</mu1>
       <mu2>0.75</mu2>
-      <fdir1>1 0 0</fdir1>
     </gazebo>
   </xacro:macro>
@@ -255,10 +266,10 @@
     <parent link="base_link"/>
     <child link="bumper_link"/>
-    <origin xyz="${chassis_length /2 + 0.12} 0.0 0.0" rpy="0.0 0.0 0.0"/>
+    <origin xyz="${chassis_length /2.0 + 0.12} 0.0 0.0" rpy="0.0 0.0 0.0"/>
   </joint>
   <!-- Chassis -->
   <link name="chassis">
     <visual>
-      <origin xyz="0 0 ${-chassis_height / 2}"/>
+      <origin xyz="0 0 ${-chassis_height / 2.0}"/>
       <geometry>
         <box size="${chassis_length} ${chassis_width} ${chassis_height}"/>
@@ -267,5 +278,5 @@
     </visual>
     <collision>
-      <origin xyz="0 0 ${-chassis_height / 2}"/>
+      <origin xyz="0 0 ${-chassis_height / 2.0}"/>
       <geometry>
         <box size="${chassis_length} ${chassis_width} ${chassis_height}"/>
@@ -275,5 +286,5 @@
         width="${chassis_length}" depth="${chassis_width}"
         height="${chassis_height}" mass="${chassis_mass}">
-      <origin xyz="0 0 ${-chassis_height / 2}"/>
+      <origin xyz="0 0 ${-chassis_height / 2.0}"/>
     </xacro:solid_cuboid_inertial>
   </link>
@@ -292,4 +303,10 @@
       <inertia ixx="0.0" ixy="0.0" ixz="0.0" iyy="0.0" iyz="0.0" izz="0.0"/>
     </inertial>
+    <collision>
+      <origin xyz="0.0 0.0 0.0" rpy="0.0 0.0 0.0"/>
+      <geometry>
+        <mesh filename="package://rr_description/urdf/assets/RR2018.stl" scale="0.0254 0.0254 0.0254"/>
+      </geometry>
+    </collision>
     <visual name="outer_shell_stl">
       <origin xyz="0.0 0.0 0.0" rpy="0.0 0.0 0.0"/>
@@ -440,10 +457,10 @@
     </gazebo>
   </xacro:macro>
-  <xacro:rr_camera name="front_facing" x_offset="0.25"
+  <xacro:rr_camera name="front_facing" x_offset="0.45"
                 y_offset="0.0" z_offset="0.29" pitch="0.0" yaw="0.0"/>
-  <xacro:rr_camera name="left_facing" x_offset="0.25"
-                y_offset="-0.15" z_offset="0.29" pitch="0.349" yaw="-0.349"/>
-  <xacro:rr_camera name="right_facing" x_offset="0.25"
-                y_offset="0.15" z_offset="0.29" pitch="0.349" yaw="0.349"/>
+  <xacro:rr_camera name="right_facing" x_offset="0.45"
+                y_offset="-0.15" z_offset="0.29" pitch="0.6" yaw="-0.6"/>
+  <xacro:rr_camera name="left_facing" x_offset="0.45"
+                y_offset="0.15" z_offset="0.29" pitch="0.6" yaw="0.6"/>
   <!-- IMU -->
   <link name="imu_link">

Commit message: update sim with new shell

File: rr_description/urdf/augmented_rc_car.urdf.xacro (robot description, xacro)
@@ -296,5 +296,5 @@
   </joint>
   <!-- Outer Shell -->
-  <!-- <link name="outer_shell">
+  <link name="outer_shell">
     <inertial>
       <origin xyz="0.0 0.0 0.0" rpy="0.0 0.0 0.0"/>
@@ -305,5 +305,5 @@
       <origin xyz="0.0 0.0 0.0" rpy="0.0 0.0 0.0"/>
       <geometry>
-        <mesh filename="package://rr_description/urdf/assets/RR2018.stl" scale="0.0254 0.0254 0.0254"/>
+        <mesh filename="package://rr_description/urdf/assets/RR2018.dae" scale="1 1 1"/>
       </geometry>
     </visual>
@@ -312,6 +312,6 @@
     <parent link="chassis"/>
     <child link="outer_shell"/>
-    <origin xyz="-0.26 -0.11 0.04" rpy="${degrees_90} 0.0 ${degrees_90}"/>
-  </joint> -->
+    <origin xyz="-0.35 -0.2 -0.2" rpy="0 0 ${degrees_90}"/>
+  </joint>
   <!-- Wheels -->
   <xacro:front_wheel lr_prefix="left" fr_prefix="front"
@@ -325,11 +325,5 @@
   <!-- Sensors -->
   <!-- Lidar -->
-  <link name="hokuyo_link">
-    <!-- <collision>
-      <origin xyz="0 0 0" rpy="0 0 0"/>
-      <geometry>
-        <box size="0.1 0.1 0.1"/>
-      </geometry>
-    </collision> -->
+  <!-- <link name="hokuyo_link">
     <inertial>
       <mass value="1e-5" />
@@ -342,5 +336,5 @@
     <parent link="chassis"/>
     <child link="hokuyo_link"/>
-  </joint>
+  </joint> -->
   <!-- ULM-30LX Hokuyo Laser Range Finder -->
   <gazebo reference="hokuyo_link">
@@ -384,9 +378,4 @@
                params="name x_offset y_offset z_offset pitch yaw">
     <link name="${name}_cam_link">
-      <visual>
-        <geometry>
-          <box size="0.05 0.05 0.05"/>
-        </geometry>
-      </visual>
       <gazebo reference="${name}_cam_link">
         <material>Gazebo/Green</material>
